File: Ortho62Unified/Ortho62Unified.kicad_pcb (KiCad board)
At the start: 2 copper layers, 179.6 x 117 mm, 81 parts, among them J1 AudioJack4, SW1 SW_Push, SW10 SW_Push, SW100 Toggle Mac/Win, SW11 SW_Push, SW12 SW_Push, SW13 SW_Push, SW14 SW_Push, SW15 SW_Push, SW16 SW_Push, SW17 SW_Push, SW18 SW_Push, SW19 SW_Push, SW2 SW_Push, SW20 SW_Push, SW21 SW_Push, SW22 SW_Push, SW23 SW_Push, SW24 SW_Push, SW25 SW_Push, SW26 SW_Push, SW27 SW_Push, SW28 SW_Push, SW29 SW_Push, SW3 SW_Push, SW30 SW_Push, SW31 SW_Push, SW32 SW_Push, SW33 SW_Push, SW4 SW_Push, SW5 SW_Push, SW6 SW_Push, SW7 SW_Push, SW8 SW_Push, SW9 SW_Push, U2 KB2040

Commit message: 66 keys placed in a grid
Parts:
- removed J1: AudioJack4, Connector_Audio:Jack_3.5mm_CUI_SJ2-3574A-SMT_Horizontal
- removed JP3: TX_RP2040, Jumper:SolderJumper-3_P1.3mm_Open_Pad1.0x1.5mm_NumberLabels
- removed JP4: RX_RP2040, Jumper:SolderJumper-3_P1.3mm_Open_Pad1.0x1.5mm_NumberLabels
- added D34: 1N4148W, Diode_SMD:D_SOD-323_Hand_Split_Keyboard, F.Cu at (158.6, 276.7)
- added D35: 1N4148W, Diode_SMD:D_SOD-323_Hand_Split_Keyboard, F.Cu at (163.7, 279.7)
- added D36: 1N4148W, Diode_SMD:D_SOD-323_Hand_Split_Keyboard, F.Cu at (163.7, 273.8)
- added D37: 1N4148W, Diode_SMD:D_SOD-323_Hand_Split_Keyboard, F.Cu at (128.3, 273.8)
- added D38: 1N4148W, Diode_SMD:D_SOD-323_Hand_Split_Keyboard, F.Cu at (148.5, 273.8)
- added D39: 1N4148W, Diode_SMD:D_SOD-323_Hand_Split_Keyboard, F.Cu at (128.3, 279.7)
- added D40: 1N4148W, Diode_SMD:D_SOD-323_Hand_Split_Keyboard, F.Cu at (133.4, 276.7)
- added D41: 1N4148W, Diode_SMD:D_SOD-323_Hand_Split_Keyboard, F.Cu at (148.5, 279.7)
- added D42: 1N4148W, Diode_SMD:D_SOD-323_Hand_Split_Keyboard, F.Cu at (143.5, 273.8)
- added D43: 1N4148W, Diode_SMD:D_SOD-323_Hand_Split_Keyboard, F.Cu at (168.7, 273.8)
- added D44: 1N4148W, Diode_SMD:D_SOD-323_Hand_Split_Keyboard, F.Cu at (133.4, 279.7)
- added D45: 1N4148W, Diode_SMD:D_SOD-323_Hand_Split_Keyboard, F.Cu at (143.5, 276.7)
- added D46: 1N4148W, Diode_SMD:D_SOD-323_Hand_Split_Keyboard, F.Cu at (123.3, 279.7)
- added D47: 1N4148W, Diode_SMD:D_SOD-323_Hand_Split_Keyboard, F.Cu at (153.6, 273.8)
- added D48: 1N4148W, Diode_SMD:D_SOD-323_Hand_Split_Keyboard, F.Cu at (123.3, 273.8)
- added D49: 1N4148W, Diode_SMD:D_SOD-323_Hand_Split_Keyboard, F.Cu at (158.6, 279.7)
- added D50: 1N4148W, Diode_SMD:D_SOD-323_Hand_Split_Keyboard, F.Cu at (168.7, 276.7)
- added D51: 1N4148W, Diode_SMD:D_SOD-323_Hand_Split_Keyboard, F.Cu at (173.8, 273.8)
- added D52: 1N4148W, Diode_SMD:D_SOD-323_Hand_Split_Keyboard, F.Cu at (148.5, 276.7)
- added D53: 1N4148W, Diode_SMD:D_SOD-323_Hand_Split_Keyboard, F.Cu at (123.3, 276.7)
- added D54: 1N4148W, Diode_SMD:D_SOD-323_Hand_Split_Keyboard, F.Cu at (158.6, 273.8)
- added D55: 1N4148W, Diode_SMD:D_SOD-323_Hand_Split_Keyboard, F.Cu at (153.6, 279.7)
- added D56: 1N4148W, Diode_SMD:D_SOD-323_Hand_Split_Keyboard, F.Cu at (138.4, 276.7)
- added D57: 1N4148W, Diode_SMD:D_SOD-323_Hand_Split_Keyboard, F.Cu at (128.3, 276.7)
- added D58: 1N4148W, Diode_SMD:D_SOD-323_Hand_Split_Keyboard, F.Cu at (138.4, 279.7)
- added D59: 1N4148W, Diode_SMD:D_SOD-323_Hand_Split_Keyboard, F.Cu at (153.6, 276.7)
- added D60: 1N4148W, Diode_SMD:D_SOD-323_Hand_Split_Keyboard, F.Cu at (118.2, 279.7)
- added D61: 1N4148W, Diode_SMD:D_SOD-323_Hand_Split_Keyboard, F.Cu at (133.4, 273.8)
- added D62: 1N4148W, Diode_SMD:D_SOD-323_Hand_Split_Keyboard, F.Cu at (118.2, 276.7)
- added D63: 1N4148W, Diode_SMD:D_SOD-323_Hand_Split_Keyboard, F.Cu at (143.5, 279.7)
- added D64: 1N4148W, Diode_SMD:D_SOD-323_Hand_Split_Keyboard, F.Cu at (163.7, 276.7)
- added D65: 1N4148W, Diode_SMD:D_SOD-323_Hand_Split_Keyboard, F.Cu at (138.4, 273.8)
- added D66: 1N4148W, Diode_SMD:D_SOD-323_Hand_Split_Keyboard, F.Cu at (118.2, 273.8)
- added SW34: SW_Push, Switch_Keyboard_Kailh:SW_Kailh_Choc_V1V2_1.00u, F.Cu at (192.5, 67.0)
- added SW35: SW_Push, Switch_Keyboard_Kailh:SW_Kailh_Choc_V1V2_1.00u, F.Cu at (212.5, 67.0)
- added SW36: SW_Push, Switch_Keyboard_Kailh:SW_Kailh_Choc_V1V2_1.00u, F.Cu at (233.5, 67.0)
- added SW37: SW_Push, Switch_Keyboard_Kailh:SW_Kailh_Choc_V1V2_1.00u, F.Cu at (254.5, 67.0)
- added SW38: SW_Push, Switch_Keyboard_Kailh:SW_Kailh_Choc_V1V2_1.00u, F.Cu at (275.5, 67.0)
- added SW39: SW_Push, Switch_Keyboard_Kailh:SW_Kailh_Choc_V1V2_1.00u, F.Cu at (296.0, 67.0)
- added SW40: SW_Push, Switch_Keyboard_Kailh:SW_Kailh_Choc_V1V2_1.50u, F.Cu at (321.0, 67.3)
- added SW41: SW_Push, Switch_Keyboard_Kailh:SW_Kailh_Choc_V1V2_1.00u, F.Cu at (192.5, 86.5)
- added SW42: SW_Push, Switch_Keyboard_Kailh:SW_Kailh_Choc_V1V2_1.00u, F.Cu at (212.5, 86.6)
- added SW43: SW_Push, Switch_Keyboard_Kailh:SW_Kailh_Choc_V1V2_1.00u, F.Cu at (233.5, 86.0)
- added SW44: SW_Push, Switch_Keyboard_Kailh:SW_Kailh_Choc_V1V2_1.00u, F.Cu at (254.5, 86.5)
- added SW45: SW_Push, Switch_Keyboard_Kailh:SW_Kailh_Choc_V1V2_1.00u, F.Cu at (275.5, 86.5)
- added SW46: SW_Push, Switch_Keyboard_Kailh:SW_Kailh_Choc_V1V2_1.00u, F.Cu at (296.0, 86.5)
- added SW47: SW_Push, Switch_Keyboard_Kailh:SW_Kailh_Choc_V1V2_1.50u, F.Cu at (321.5, 124.0)
- added SW48: SW_Push, Switch_Keyboard_Kailh:SW_Kailh_Choc_V1V2_1.00u, F.Cu at (192.5, 106.0)
- added SW49: SW_Push, Switch_Keyboard_Kailh:SW_Kailh_Choc_V1V2_1.00u, F.Cu at (212.5, 106.0)
- added SW50: SW_Push, Switch_Keyboard_Kailh:SW_Kailh_Choc_V1V2_1.00u, F.Cu at (233.5, 105.5)
- added SW51: SW_Push, Switch_Keyboard_Kailh:SW_Kailh_Choc_V1V2_1.00u, F.Cu at (254.5, 106.5)
- added SW52: SW_Push, Switch_Keyboard_Kailh:SW_Kailh_Choc_V1V2_1.00u, F.Cu at (275.5, 106.0)
- added SW53: SW_Push, Switch_Keyboard_Kailh:SW_Kailh_Choc_V1V2_1.00u, F.Cu at (296.0, 106.0)
- added SW54: SW_Push, Switch_Keyboard_Kailh:SW_Kailh_Choc_V1V2_1.50u, F.Cu at (321.0, 105.5)
- added SW55: SW_Push, Switch_Keyboard_Kailh:SW_Kailh_Choc_V1V2_1.00u, F.Cu at (192.5, 125.5)
- added SW56: SW_Push, Switch_Keyboard_Kailh:SW_Kailh_Choc_V1V2_1.00u, F.Cu at (212.5, 125.5)
- added SW57: SW_Push, Switch_Keyboard_Kailh:SW_Kailh_Choc_V1V2_1.00u, F.Cu at (233.5, 125.0)
- added SW58: SW_Push, Switch_Keyboard_Kailh:SW_Kailh_Choc_V1V2_1.00u, F.Cu at (254.5, 126.5)
- added SW59: SW_Push, Switch_Keyboard_Kailh:SW_Kailh_Choc_V1V2_1.00u, F.Cu at (275.5, 125.5)
- added SW60: SW_Push, Switch_Keyboard_Kailh:SW_Kailh_Choc_V1V2_1.00u, F.Cu at (296.0, 125.5)
- added SW61: SW_Push, Switch_Keyboard_Kailh:SW_Kailh_Choc_V1V2_1.50u, F.Cu at (321.0, 86.4)
- added SW62: SW_Push, Switch_Keyboard_Kailh:SW_Kailh_Choc_V1V2_1.00u, F.Cu at (212.5, 144.5)
- added SW63: SW_Push, Switch_Keyboard_Kailh:SW_Kailh_Choc_V1V2_1.00u, F.Cu at (233.5, 144.5)
- added SW64: SW_Push, Switch_Keyboard_Kailh:SW_Kailh_Choc_V1V2_1.00u, F.Cu at (254.5, 146.5)
- added SW65: SW_Push, Switch_Keyboard_Kailh:SW_Kailh_Choc_V1V2_1.00u, F.Cu at (275.5, 145.0)
- added SW66: SW_Push, Switch_Keyboard_Kailh:SW_Kailh_Choc_V1V2_1.00u, F.Cu at (296.0, 144.5)
- SW1, SW10, SW11, SW12, SW13, SW14, SW15, SW16, SW17, SW18, SW19, SW2, SW20, SW21, SW22, SW23, SW24, SW26, SW27, SW28, SW3, SW30, SW4, SW5, SW6, SW7, SW8, SW9: footprint Lily58-footprint:MX_PG1350-DoubleSide_Keycap_18mm_1.00u -> Switch_Keyboard_Kailh:SW_Kailh_Choc_V1V2_1.00u
- SW25, SW31, SW32, SW33: footprint Lily58-footprint:MX_PG1350-DoubleSide_Keycap_28mm_1.50u -> Switch_Keyboard_Kailh:SW_Kailh_Choc_V1V2_1.50u
- SW29: footprint Lily58-footprint:MX_PG1350-DoubleSide_Keycap_28mm_1.50u -> Switch_Keyboard_Kailh:SW_Kailh_Choc_V1V2_1.00u
- moved D32 81.5 mm to (143.0, 141.0)
- moved SW29 81.5 mm to (151.2, 146.0)
- moved D33 76.6 mm to (162.9, 140.8)
- moved SW30 76.6 mm to (171.0, 146.0)
- moved H3 71.9 mm to (177.5, 21.1), turned to 90 degrees
- moved D29 68.6 mm to (85.9, 140.4)
- moved D30 68.6 mm to (103.2, 141.2)
- moved D31 68.6 mm to (123.2, 141.0)
- moved SW26 68.6 mm to (91.4, 146.0)
- moved SW27 68.6 mm to (111.5, 146.0)
- moved SW28 68.6 mm to (131.2, 146.0)
- moved C1 59.8 mm to (184.0, 27.1), turned to 0 degrees
- moved SW100 57.7 mm to (228.0, 29.1), turned to -90 degrees
- moved R1 56.5 mm to (192.5, 25.6), turned to 180 degrees
- moved D22 54.0 mm to (63.8, 121.5), turned to -90 degrees
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Routing:
- removed copper zone on B.Cu, net GND
- removed copper zone on F.Cu, net GND
Other:
- board outline removed

Commit message: 66 keys in grid
Parts:
- moved SW61 131.1 mm to (203.5, 144.5)
- moved SW62 15.5 mm to (228.0, 144.5)
- moved SW63 15.5 mm to (249.0, 144.5)
- moved SW64 15.5 mm to (270.0, 146.5)
- moved SW65 15.5 mm to (291.0, 145.0)
- moved SW66 15.5 mm to (311.5, 144.5)
- moved D29 12.0 mm to (73.9, 140.4)
- moved D30 12.0 mm to (91.2, 141.2)
- moved D31 12.0 mm to (111.2, 141.0)
- moved D32 12.0 mm to (131.0, 141.0)
- moved D33 12.0 mm to (150.9, 140.8)
- moved SW26 12.0 mm to (79.4, 146.0)
- moved SW27 12.0 mm to (99.5, 146.0)
- moved SW28 12.0 mm to (119.2, 146.0)
- moved SW29 12.0 mm to (139.2, 146.0)
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Changed lines of the file:
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@@
   )
   (footprint "Switch_Keyboard_Kailh:SW_Kailh_Choc_V1V2_1.00u" (layer "F.Cu")
-    (at 233.5 144.5)
+    (at 249 144.5)
     (descr "Kailh Choc keyswitch CPG1350 V1 CPG1353 V2 with 1.00u keycap")
     (tags "Kailh Choc Keyswitch Switch CPG1350 V1 CPG1353 V2 Cutout 1.00u")
@@
   )
   (footprint "Switch_Keyboard_Kailh:SW_Kailh_Choc_V1V2_1.00u" (layer "F.Cu")
-    (at 151.25 145.979185)
+    (at 139.25 145.979185)
     (descr "Kailh Choc keyswitch CPG1350 V1 CPG1353 V2 with 1.00u keycap")
     (tags "Kailh Choc Keyswitch Switch CPG1350 V1 CPG1353 V2 Cutout 1.00u")
@@
   )
   (footprint "Switch_Keyboard_Kailh:SW_Kailh_Choc_V1V2_1.00u" (layer "F.Cu")
-    (at 254.5 146.5)
+    (at 270 146.5)
     (descr "Kailh Choc keyswitch CPG1350 V1 CPG1353 V2 with 1.00u keycap")
     (tags "Kailh Choc Keyswitch Switch CPG1350 V1 CPG1353 V2 Cutout 1.00u")
@@
   )
   (footprint "Switch_Keyboard_Kailh:SW_Kailh_Choc_V1V2_1.00u" (layer "F.Cu")
-    (at 111.5 146.004185)
+    (at 99.5 146.004185)
     (descr "Kailh Choc keyswitch CPG1350 V1 CPG1353 V2 with 1.00u keycap")
     (tags "Kailh Choc Keyswitch Switch CPG1350 V1 CPG1353 V2 Cutout 1.00u")
@@
   )
   (footprint "Switch_Keyboard_Kailh:SW_Kailh_Choc_V1V2_1.00u" (layer "F.Cu")
-    (at 275.5 145)
+    (at 291 145)
     (descr "Kailh Choc keyswitch CPG1350 V1 CPG1353 V2 with 1.00u keycap")
     (tags "Kailh Choc Keyswitch Switch CPG1350 V1 CPG1353 V2 Cutout 1.00u")
@@
   )
   (footprint "Switch_Keyboard_Kailh:SW_Kailh_Choc_V1V2_1.00u" (layer "F.Cu")
-    (at 296 144.5)
+    (at 311.5 144.5)
     (descr "Kailh Choc keyswitch CPG1350 V1 CPG1353 V2 with 1.00u keycap")
     (tags "Kailh Choc Keyswitch Switch CPG1350 V1 CPG1353 V2 Cutout 1.00u")
@@
   )
   (footprint "Switch_Keyboard_Kailh:SW_Kailh_Choc_V1V2_1.00u" (layer "F.Cu")
-    (at 171 146)
+    (at 159 146)
     (descr "Kailh Choc keyswitch CPG1350 V1 CPG1353 V2 with 1.00u keycap")
     (tags "Kailh Choc Keyswitch Switch CPG1350 V1 CPG1353 V2 Cutout 1.00u")
@@
   )
   (footprint "Switch_Keyboard_Kailh:SW_Kailh_Choc_V1V2_1.50u" (layer "F.Cu")
-    (at 321 86.38)
+    (at 203.5 144.5)
     (descr "Kailh Choc keyswitch CPG1350 V1 CPG1353 V2 with 1.50u keycap")
     (tags "Kailh Choc Keyswitch Switch CPG1350 V1 CPG1353 V2 Cutout 1.50u")
@@
   )
   (footprint "Switch_Keyboard_Kailh:SW_Kailh_Choc_V1V2_1.00u" (layer "F.Cu")
-    (at 212.5 144.5)
+    (at 228 144.5)
     (descr "Kailh Choc keyswitch CPG1350 V1 CPG1353 V2 with 1.00u keycap")
     (tags "Kailh Choc Keyswitch Switch CPG1350 V1 CPG1353 V2 Cutout 1.00u")
@@
   )
   (footprint "Switch_Keyboard_Kailh:SW_Kailh_Choc_V1V2_1.00u" (layer "F.Cu")
-    (at 131.25 146.004185)
+    (at 119.25 146.004185)
     (descr "Kailh Choc keyswitch CPG1350 V1 CPG1353 V2 with 1.00u keycap")
     (tags "Kailh Choc Keyswitch Switch CPG1350 V1 CPG1353 V2 Cutout 1.00u")
@@
   )
   (footprint "Switch_Keyboard_Kailh:SW_Kailh_Choc_V1V2_1.00u" (layer "F.Cu")
-    (at 91.4 145.979185)
+    (at 79.4 145.979185)
     (descr "Kailh Choc keyswitch CPG1350 V1 CPG1353 V2 with 1.00u keycap")
     (tags "Kailh Choc Keyswitch Switch CPG1350 V1 CPG1353 V2 Cutout 1.00u")
@@
   )
   (footprint "Diode_SMD:D_SOD-323_Hand_Split_Keyboard" (layer "B.Cu")
-    (at 85.9 140.379185 90)
+    (at 73.9 140.379185 90)
     (descr "SOD-323")
     (tags "SOD-323")
@@
   )
   (footprint "Diode_SMD:D_SOD-323_Hand_Split_Keyboard" (layer "B.Cu")
-    (at 103.25 141.229185 -90)
+    (at 91.25 141.229185 -90)
     (descr "SOD-323")
     (tags "SOD-323")
@@
   )
   (footprint "Diode_SMD:D_SOD-323_Hand_Split_Keyboard" (layer "B.Cu")
-    (at 143 140.979185 -90)
+    (at 131 140.979185 -90)
     (descr "SOD-323")
     (tags "SOD-323")
@@
   )
   (footprint "Diode_SMD:D_SOD-323_Hand_Split_Keyboard" (layer "B.Cu")
-    (at 123.25 140.979185 -90)
+    (at 111.25 140.979185 -90)
     (descr "SOD-323")
     (tags "SOD-323")
@@
   )
   (footprint "Diode_SMD:D_SOD-323_Hand_Split_Keyboard" (layer "B.Cu")
-    (at 162.9 140.75 -89.99999997)
+    (at 150.9 140.75 -89.99999997)
     (descr "SOD-323")
     (tags "SOD-323")

Commit message: Connections for grid layout keys.
Parts:
- removed JP1: Left/Right, Jumper:SolderJumper-2_P1.3mm_Open_TrianglePad1.0x1.5mm
- removed JP2: Choice, Jumper:SolderJumper-2_P1.3mm_Open_TrianglePad1.0x1.5mm
- removed SW100: Toggle Mac/Win, Button_Switch_SMD:SW_SPST_CK_RS282G05A3
- added C10: 100n, Capacitor_SMD:C_0603_1608Metric, F.Cu at (371.3, 44.8)
- added C11: 100n, Capacitor_SMD:C_0603_1608Metric, F.Cu at (359.3, 45.5)
- added C12: 1u, Capacitor_SMD:C_0603_1608Metric, F.Cu at (363.3, 44.8)
- added C13: 1u, Capacitor_SMD:C_0603_1608Metric, F.Cu at (375.0, 38.0)
- added C2: 1u, Capacitor_SMD:C_0603_1608Metric, F.Cu at (367.3, 44.8)
- added C3: 100n, Capacitor_SMD:C_0603_1608Metric, F.Cu at (379.0, 33.0)
- added C4: 100n, Capacitor_SMD:C_0603_1608Metric, F.Cu at (368.0, 42.3)
- added C5: 100n, Capacitor_SMD:C_0603_1608Metric, F.Cu at (355.3, 45.5)
- added C6: 100n, Capacitor_SMD:C_0603_1608Metric, F.Cu at (360.0, 42.3)
- added C7: 100n, Capacitor_SMD:C_0603_1608Metric, F.Cu at (379.0, 38.0)
- added C8: 100n, Capacitor_SMD:C_0603_1608Metric, F.Cu at (375.0, 33.0)
- added C9: 100n, Capacitor_SMD:C_0603_1608Metric, F.Cu at (364.0, 42.3)
- added J1: USB_B_Micro, Connector_USB:USB_Micro-B_Molex_47346-0001, F.Cu at (358.5, 34.9)
- added R2: 27.4, Resistor_SMD:R_0603_1608Metric, F.Cu at (372.0, 42.3)
- added U1: MCP1700T-3302E_TT, digikey-footprints:SOT-23-3, F.Cu at (355.6, 41.8)
- C1: value C -> 1u
- R1: value 0 -> 27.4; footprint Resistor_SMD:R_0603_1608Metric_Pad0.98x0.95mm_HandSolder -> Resistor_SMD:R_0603_1608Metric; moved to F.Cu
- SW30: footprint Switch_Keyboard_Kailh:SW_Kailh_Choc_V1V2_1.00u -> Switch_Keyboard_Kailh:SW_Kailh_Choc_V1V2_1.50u
- U2: value KB2040 -> RP2040; footprint KB2040:Adafruit_KB2040 -> Package_DFN_QFN:QFN-56-1EP_7x7mm_P0.4mm_EP3.2x3.2mm
- moved C1 191.2 mm to (375.0, 35.5)
- moved R1 186.8 mm to (379.0, 35.5), turned to 0 degrees
- moved U2 177.3 mm to (368.4, 36.4), turned to 0 degrees
- moved D9 68.0 mm to (72.0, 167.5)
- moved D16 64.6 mm to (80.5, 168.4)
- moved D17 64.6 mm to (99.7, 168.4)
- moved D18 64.6 mm to (118.9, 168.5)
- moved D19 64.6 mm to (138.1, 165.6)
- moved D20 64.6 mm to (157.3, 168.7)
- moved D21 64.6 mm to (176.5, 168.5)
- moved D22 55.9 mm to (78.7, 175.3)
- moved D23 55.9 mm to (98.4, 175.3)
- moved D24 55.9 mm to (116.1, 180.0)
- moved D25 55.9 mm to (135.3, 180.0)
- moved D26 55.9 mm to (155.3, 180.0)
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Connections:
- C1 pad 1: +VDC -> +1V1
- C1 pad 2: GND -> +1V1
- R1 pad 1: Net-(R1-Pad1) -> /USB_D+
- R1 pad 2: +VDC -> /USB_DP
- U2 pad 1: unconnected-(U2-Pad1) -> +3V3
- U2 pad 10: Net-(JP2-Pad2) -> +3V3
- U2 pad 11: /ROW_4 -> unconnected-(U2-Pad11)
- U2 pad 12: /ROW_3 -> unconnected-(U2-Pad12)
- U2 pad 13: /ROW_2 -> unconnected-(U2-Pad13)
- U2 pad 14: /ROW_1 -> unconnected-(U2-Pad14)
- U2 pad 15: /ROW_0 -> unconnected-(U2-Pad15)
- U2 pad 16: /COL_5 -> unconnected-(U2-Pad16)
- U2 pad 17: /COL_4 -> unconnected-(U2-Pad17)
- U2 pad 18: /COL_3 -> unconnected-(U2-Pad18)
- U2 pad 19: /COL_2 -> unconnected-(U2-Pad19)
- U2 pad 2: /UART0_TX -> unconnected-(U2-Pad2)
- U2 pad 20: /COL_1 -> unconnected-(U2-Pad20)
- U2 pad 21: /COL_0 -> unconnected-(U2-Pad21)
- U2 pad 22: unconnected-(U2-Pad22) -> +3V3
- U2 pad 23: unconnected-(U2-Pad23) -> +1V1
- U2 pad 24: GND -> unconnected-(U2-Pad24)
- U2 pad 25: Net-(R1-Pad1) -> unconnected-(U2-Pad25)
- U2 pad 3: /UART0_RX -> unconnected-(U2-Pad3)
- U2 pad 4: GND -> unconnected-(U2-Pad4)
- U2 pad 5: GND -> unconnected-(U2-Pad5)
- U2 pad 6: /I2C1_SCK -> unconnected-(U2-Pad6)
- U2 pad 7: /I2C1_SDA -> unconnected-(U2-Pad7)
- U2 pad 8: Net-(SW100-Pad2) -> unconnected-(U2-Pad8)
- U2 pad 9: Net-(JP1-Pad2) -> unconnected-(U2-Pad9)
