File: Ortho62Unified/Ortho62Unified.kicad_sch (KiCad schematic)
At the start: 81 parts, among them J1 AudioJack4, SW1 SW_Push, SW10 SW_Push, SW100 Toggle Mac/Win, SW11 SW_Push, SW12 SW_Push, SW13 SW_Push, SW14 SW_Push, SW15 SW_Push, SW16 SW_Push, SW17 SW_Push, SW18 SW_Push, SW19 SW_Push, SW2 SW_Push, SW20 SW_Push, SW21 SW_Push, SW22 SW_Push, SW23 SW_Push, SW24 SW_Push, SW25 SW_Push, SW26 SW_Push, SW27 SW_Push, SW28 SW_Push, SW29 SW_Push, SW3 SW_Push, SW30 SW_Push, SW31 SW_Push, SW32 SW_Push, SW33 SW_Push, SW4 SW_Push, SW5 SW_Push, SW6 SW_Push, SW7 SW_Push, SW8 SW_Push, SW9 SW_Push, U2 KB2040

Commit message: 66 keys placed in a grid
Parts:
- removed J1: AudioJack4, Connector_Audio:Jack_3.5mm_CUI_SJ2-3574A-SMT_Horizontal, symbol Connector:AudioJack4
- removed JP3: TX_RP2040, Jumper:SolderJumper-3_P1.3mm_Open_Pad1.0x1.5mm_NumberLabels, symbol Jumper:SolderJumper_3_Open
- removed JP4: RX_RP2040, Jumper:SolderJumper-3_P1.3mm_Open_Pad1.0x1.5mm_NumberLabels, symbol Jumper:SolderJumper_3_Open
- added D34, D35, D36, D37, D38, D39, D40, D41, D42, D43, D44, D45, D46, D47, D48, D49, D50, D51, D52, D53, D54, D55, D56, D57, D58, D59, D60, D61, D62, D63, D64, D65, D66: 1N4148W, Diode_SMD:D_SOD-323_Hand_Split_Keyboard, symbol Diode:1N4148W
- added SW34, SW35, SW36, SW37, SW38, SW39, SW41, SW42, SW43, SW44, SW45, SW46, SW48, SW49, SW50, SW51, SW52, SW53, SW55, SW56, SW57, SW58, SW59, SW60, SW62, SW63, SW64, SW65, SW66: SW_Push, Switch_Keyboard_Kailh:SW_Kailh_Choc_V1V2_1.00u, symbol Switch:SW_Push
- added SW40, SW47, SW54, SW61: SW_Push, Switch_Keyboard_Kailh:SW_Kailh_Choc_V1V2_1.50u, symbol Switch:SW_Push
- SW1, SW10, SW11, SW12, SW13, SW14, SW15, SW16, SW17, SW18, SW19, SW2, SW20, SW21, SW22, SW23, SW24, SW26, SW27, SW28, SW3, SW30, SW4, SW5, SW6, SW7, SW8, SW9: footprint Lily58-footprint:MX_PG1350-DoubleSide_Keycap_18mm_1.00u -> Switch_Keyboard_Kailh:SW_Kailh_Choc_V1V2_1.00u
- SW25, SW31, SW32, SW33: footprint Lily58-footprint:MX_PG1350-DoubleSide_Keycap_28mm_1.50u -> Switch_Keyboard_Kailh:SW_Kailh_Choc_V1V2_1.50u
- SW29: footprint Lily58-footprint:MX_PG1350-DoubleSide_Keycap_28mm_1.50u -> Switch_Keyboard_Kailh:SW_Kailh_Choc_V1V2_1.00u
Connections:
- net ROW_0: now also D34.1 (K), D35.1 (K), D36.1 (K), D37.1 (K), D38.1 (K), D39.1 (K), D40.1 (K)
- net ROW_1: now also D41.1 (K), D42.1 (K), D43.1 (K), D44.1 (K), D45.1 (K), D46.1 (K), D47.1 (K)
- net ROW_2: now also D48.1 (K), D49.1 (K), D50.1 (K), D51.1 (K), D52.1 (K), D53.1 (K), D54.1 (K)
- net ROW_3: now also D55.1 (K), D56.1 (K), D57.1 (K), D58.1 (K), D59.1 (K), D60.1 (K)
- net ROW_4: now also D61.1 (K), D62.1 (K), D63.1 (K), D64.1 (K), D65.1 (K), D66.1 (K)
- new net: D49.2 (A), SW49.2
- new net: D48.2 (A), SW48.2
- new net: D44.2 (A), SW44.2
- new net: D35.2 (A), SW35.2
- new net: D36.2 (A), SW36.2
- new net: D51.2 (A), SW51.2
- new net: D34.2 (A), SW34.2
- new net: D54.2 (A), SW54.2
- new net: D64.2 (A), SW64.2
- new net: D47.2 (A), SW47.2
- new net: D43.2 (A), SW43.2
- new net: D41.2 (A), SW41.2
- new net: D37.2 (A), SW37.2
- new net: D45.2 (A), SW45.2
- new net: D52.2 (A), SW52.2
- new net: D63.2 (A), SW63.2
- new net: D56.2 (A), SW56.2
- new net: D42.2 (A), SW42.2
- new net: D65.2 (A), SW65.2
- new net: D58.2 (A), SW58.2
- new net: D57.2 (A), SW57.2
- new net: D62.2 (A), SW62.2
- new net: D61.2 (A), SW61.2
- new net: D66.2 (A), SW66.2
- new net: D59.2 (A), SW59.2
- new net: D46.2 (A), SW46.2
- new net: D60.2 (A), SW60.2
- new net: D50.2 (A), SW50.2
- new net: D55.2 (A), SW55.2
- new net: D53.2 (A), SW53.2
- new net: D40.2 (A), SW40.2
- new net: D39.2 (A), SW39.2
- new net: D38.2 (A), SW38.2
- new net COL_10: SW37.1, SW44.1, SW51.1, SW58.1, SW64.1
- new net COL_11: SW38.1, SW45.1, SW52.1, SW59.1, SW65.1
- new net COL_12: SW39.1, SW46.1, SW53.1, SW60.1, SW66.1
- new net COL_13: SW40.1, SW47.1, SW54.1
- new net COL_7: SW34.1, SW41.1, SW48.1, SW55.1, SW61.1
- new net COL_8: SW35.1, SW42.1, SW49.1, SW56.1, SW62.1
- new net COL_9: SW36.1, SW43.1, SW50.1, SW57.1, SW63.1
Other:
- title: Mac 60 Keys Split Keyboard -> 66 Keys Ortholinear Keyboard
- moved on the sheet: C1, H2, H3, H4, H5, H6, H7, JP1, JP2, R1, SW100, U2

Commit message: 66 keys in grid
Parts:
- SW30: footprint Switch_Keyboard_Kailh:SW_Kailh_Choc_V1V2_1.00u -> Switch_Keyboard_Kailh:SW_Kailh_Choc_V1V2_1.50u
Changed lines of the file:
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@@
     (property "Reference" "SW30" (id 0) (at 130.175 134.62 0))
     (property "Value" "SW_Push" (id 1) (at 130.175 137.16 0))
-    (property "Footprint" "Switch_Keyboard_Kailh:SW_Kailh_Choc_V1V2_1.00u" (id 2) (at 130.175 137.16 0)
+    (property "Footprint" "Switch_Keyboard_Kailh:SW_Kailh_Choc_V1V2_1.50u" (id 2) (at 130.175 137.16 0)
       (effects (font (size 1.27 1.27)) hide)
     )
@@
     )
     (path "/cf30b61b-518f-4fc0-9759-5e2e77a579bf"
-      (reference "SW30") (unit 1) (value "SW_Push") (footprint "Switch_Keyboard_Kailh:SW_Kailh_Choc_V1V2_1.00u")
+      (reference "SW30") (unit 1) (value "SW_Push") (footprint "Switch_Keyboard_Kailh:SW_Kailh_Choc_V1V2_1.50u")
     )
     (path "/73eae815-5b46-42a8-bd47-b5e4553af68e"

Commit message: Connections for grid layout keys.
Parts:
- removed JP1: Left/Right, Jumper:SolderJumper-2_P1.3mm_Open_TrianglePad1.0x1.5mm, symbol Jumper:SolderJumper_2_Open
- removed JP2: Choice, Jumper:SolderJumper-2_P1.3mm_Open_TrianglePad1.0x1.5mm, symbol Jumper:SolderJumper_2_Open
- removed SW100: Toggle Mac/Win, Button_Switch_SMD:SW_SPST_CK_RS282G05A3, symbol Switch:SW_SPST
- removed U2: KB2040, KB2040:Adafruit_KB2040, symbol KB2040:KB2040
- added C10, C11, C3, C4, C5, C6, C7, C8, C9: 100n, Capacitor_SMD:C_0603_1608Metric, symbol Device:C
- added C12, C13, C2: 1u, Capacitor_SMD:C_0603_1608Metric, symbol Device:C
- added J1: USB_B_Micro, Connector_USB:USB_Micro-B_Molex_47346-0001, symbol Connector:USB_B_Micro
- added R2: 27.4, Resistor_SMD:R_0603_1608Metric, symbol Device:R
- added U1: MCP1700T-3302E_TT, digikey-footprints:SOT-23-3, symbol dk_PMIC-Voltage-Regulators-Linear:MCP1700T-3302E_TT
- added U2: RP2040, Package_DFN_QFN:QFN-56-1EP_7x7mm_P0.4mm_EP3.2x3.2mm, symbol MCU_RaspberryPi:RP2040
- C1: value C -> 1u
- R1: value 0 -> 27.4; footprint Resistor_SMD:R_0603_1608Metric_Pad0.98x0.95mm_HandSolder -> Resistor_SMD:R_0603_1608Metric
Connections:
- net GND: now also C12.2, C13.2, C3.2, C4.2, J1.5 (GND), U1.1 (GND); no longer C1.2
- net USB_D+: now reaches R1.1
- net USB_D+: now also J1.3 (D+)
- net +VDC renamed +1V1
- net +1V1: now also C1.2, C3.1, C4.1, U2.23 (DVDD), U2.45 (VREG_VOUT), U2.50 (DVDD); no longer R1.2
- new net: C10.2, C11.2, C2.2, C5.2, C6.2, C7.2, C8.2, C9.2
- new net: C12.1, J1.1 (VBUS), U1.3 (IN)
- new net +3V3: C10.1, C11.1, C13.1, C2.1, C5.1, C6.1, C7.1, C8.1, C9.1, U1.2 (OUT), U2.1 (IOVDD), U2.10 (IOVDD), U2.22 (IOVDD), U2.33 (IOVDD), U2.42 (IOVDD), U2.43 (ADC_AVDD), U2.44 (VREG_IN), U2.48 (USB_VDD), U2.49 (IOVDD)
- new net USB_D-: J1.2 (D-), R2.1
- new net USB_DM: R2.2, U2.46 (USB_DM)
- new net USB_DP: R1.2, U2.47 (USB_DP)
- no-connect marks 2 -> 0
Other:
- note added: "Must be close to pin 44"
- note added: "Must be close to pin 45"
- moved on the sheet: H2, H3, H4, H5, H6, H7
