File: MacSplitNN/MacSplit60.kicad_sch (KiCad schematic)
At the start: 73 parts, among them J1 USB_C_Receptacle_USB2.0, SW1 SW_Push, SW10 SW_Push, SW100 SW_SPST, SW11 SW_Push, SW12 SW_Push, SW13 SW_Push, SW14 SW_Push, SW15 SW_Push, SW16 SW_Push, SW17 SW_Push, SW18 SW_Push, SW19 SW_Push, SW2 SW_Push, SW20 SW_Push, SW21 SW_Push, SW22 SW_Push, SW23 SW_Push, SW24 SW_Push, SW25 SW_Push, SW26 SW_Push, SW27 SW_Push, SW28 SW_Push, SW29 SW_Push, SW3 SW_Push, SW30 SW_Push, SW4 SW_Push, SW5 SW_Push, SW6 SW_Push, SW7 SW_Push, SW8 SW_Push, SW9 SW_Push, U1 Pico, U2 MCP23S17_ML

Commit message: Draft update - remove USB-C and IO Expander chip, unroute all.
Parts:
- removed J1: USB_C_Receptacle_USB2.0, Connector_USB:USB_C_Receptacle_GCT_USB4085_Circular, symbol Connector:USB_C_Receptacle_USB2.0
- removed U2: MCP23S17_ML, Package_DFN_QFN:QFN-28-1EP_6x6mm_P0.65mm_EP4.25x4.25mm, symbol Interface_Expansion:MCP23S17_ML
- added A1: Adafruit_Feather_Generic, Module:Adafruit_Feather, symbol MCU_Module:Adafruit_Feather_Generic
- added J1: Conn_01x04_Pin, Connector_JST:JST_PH_S4B-PH-SM4-TB_1x04-1MP_P2.00mm_Horizontal, symbol Connector:Conn_01x04_Pin
- added U3: MCP23017_SO, Package_SO:SOIC-28W_7.5x17.9mm_P1.27mm, symbol Interface_Expansion:MCP23017_SO
Connections:
- net +VDC: now also J1.1 (Pin_1), U3.18 (~{RESET}), U3.9 (VDD)
- net COL_0: now also U3.21 (GPA0)
- net COL_1: now also U3.22 (GPA1)
- net COL_2: now also U3.23 (GPA2)
- net COL_3: now also U3.24 (GPA3)
- net COL_4: now also U3.25 (GPA4)
- net COL_5: now also U3.26 (GPA5)
- net GND: now also J1.4 (Pin_4), U3.10 (VSS), U3.15 (A0), U3.16 (A1), U3.17 (A2)
- net ROW_0: now also U3.1 (GPB0)
- net ROW_1: now also U3.2 (GPB1)
- net ROW_2: now also U3.3 (GPB2)
- net ROW_3: now also U3.4 (GPB3)
- net ROW_4: now also U3.5 (GPB4)
- net SPI0_CSn: no longer names the net of U1.7 (GPIO5)
- net SPI0_RX: no longer names the net of U1.6 (GPIO4)
- net SPI0_SCK renamed SDA_IOEXP
- net SDA_IOEXP: now also J1.2 (Pin_2), U3.13 (SDA)
- net SPI0_TX renamed SCL_IOEXP
- net SCL_IOEXP: now also J1.3 (Pin_3), U3.12 (SCK)
