File: Ortho82Split/Ortho82Split/Ortho82Split.kicad_pcb (KiCad board)
At the start: 2 copper layers, 147.9 x 134.5 mm, 153 parts, among them J1 Left-Right, J3 USB_C_Receptacle_USB2.0, J9 TC2030-IDC-NL, SW11 SW_Push, SW12 SW_Push, SW13 SW_Push, SW14 SW_Push, SW15 SW_Push, SW16 SW_Push, SW17 SW_Push, SW18 SW_Push, SW19 SW_Push, SW20 SW_Push, SW21 SW_Push, SW22 SW_Push, SW23 SW_Push, SW24 SW_Push, SW25 SW_Push, SW26 SW_Push, SW27 SW_Push, SW28 SW_Push, SW29 SW_Push, SW30 SW_Push, SW31 SW_Push, SW32 SW_Push, SW33 SW_Push, SW34 SW_Push, SW35 SW_Push, SW36 SW_Push, SW37 SW_Push, SW38 SW_Push, SW39 SW_Push, SW40 SW_Push, SW41 SW_Push, SW42 SW_Push, SW43 SW_Push, SW44 SW_Push, SW45 SW_Push, SW46 SW_Push, SW47 SW_Push, SW48 SW_Push, SW49 SW_Push, SW50 SW_Push, SW51 SW_Push, SW74 Left/Right, SW83 ~{RESET}, U1 MCP1700T-3302E_TT, U2 ATxmega32A4U-A, U3 USBLC6-2SC6

Commit message: Correct spacing and kb2040 try.
Parts:
- removed 0402: C_0402_1005Metric, Capacitor_SMD:C_0402_1005Metric
- removed 0603: C_0603_1608Metric, Capacitor_SMD:C_0603_1608Metric
- removed 0805: C_0805_2012Metric, Capacitor_SMD:C_0805_2012Metric
- removed 1.27: PinHeader_1x06_P1.27mm_Vertical, Connector_PinHeader_1.27mm:PinHeader_1x06_P1.27mm_Vertical
- removed 1206: C_1206_3216Metric, Capacitor_SMD:C_1206_3216Metric
- removed 1210: C_1210_3225Metric, Capacitor_SMD:C_1210_3225Metric
- removed 1812: C_1812_4532Metric, Capacitor_SMD:C_1812_4532Metric
- removed 1mm: PinHeader_1x08_P1.00mm_Vertical, Connector_PinHeader_1.00mm:PinHeader_1x08_P1.00mm_Vertical
- removed 2.54: PinHeader_1x04_P2.54mm_Vertical, Connector_PinHeader_2.54mm:PinHeader_1x04_P2.54mm_Vertical
- removed 2mm: PinHeader_1x05_P2.00mm_Vertical, Connector_PinHeader_2.00mm:PinHeader_1x05_P2.00mm_Vertical
- removed 3214G: Potentiometer_Bourns_3214G_Horizontal, Potentiometer_SMD:Potentiometer_Bourns_3214G_Horizontal
- removed 3224W: Potentiometer_Bourns_3224W_Vertical, Potentiometer_SMD:Potentiometer_Bourns_3224W_Vertical
- removed 3314R: Potentiometer_Bourns_3314R-GM5_Vertical, Potentiometer_SMD:Potentiometer_Bourns_3314R-GM5_Vertical
- removed 6.3x5.4: CP_Elec_6.3x5.4_Nichicon, Capacitor_SMD:CP_Elec_6.3x5.4_Nichicon
- removed C1, C2, C6, C7: 100n, Capacitor_SMD:C_0603_1608Metric_Pad1.08x0.95mm_HandSolder
- removed C3, C4, C5: 1u, Capacitor_SMD:C_0603_1608Metric_Pad1.08x0.95mm_HandSolder
- removed the D38 at (59.8, 167.3)
- removed D41: 1N4148W, HandsolderModifiedComponents:D_SOD-123F_DoubleSided
- removed D76: Red, LED_THT:LED_D3.0mm
- removed F1: Polyfuse, Fuse:Fuse_1206_3216Metric_Pad1.42x1.75mm_HandSolder
- removed FID1, FID2, FID3: Fiducial, Fiducial:Fiducial_0.5mm_Mask1mm
- removed J1: Left-Right, Connector_PinHeader_2.00mm:PinHeader_1x04_P2.00mm_Vertical
- removed J3: USB_C_Receptacle_USB2.0, CustomHandSolderConnectors:USB_C_Receptacle_GCT_USB4085_HandSolder_SMT
- removed J9: TC2030-IDC-NL, Tag_Connect:TC2030-IDC-NL
- removed LQFP48: LQFP-48-1EP_7x7mm_P0.5mm_EP3.6x3.6mm, Package_QFP:LQFP-48-1EP_7x7mm_P0.5mm_EP3.6x3.6mm
- removed MSOP-8: MSOP-8-1EP_3x3mm_P0.65mm_EP1.68x1.88mm, Package_SO:MSOP-8-1EP_3x3mm_P0.65mm_EP1.68x1.88mm
- removed MSOP16: MSOP-16-1EP_3x4.039mm_P0.5mm_EP1.651x2.845mm, Package_SO:MSOP-16-1EP_3x4.039mm_P0.5mm_EP1.651x2.845mm
- removed PLCC6: LED_RGB_PLCC-6, LED_SMD:LED_RGB_PLCC-6
- removed QFN32: QFN-32-1EP_5x5mm_P0.5mm_EP3.1x3.1mm, Package_DFN_QFN:QFN-32-1EP_5x5mm_P0.5mm_EP3.1x3.1mm
- removed QFN48: QFN-48-1EP_7x7mm_P0.5mm_EP5.3x5.3mm, Package_DFN_QFN:QFN-48-1EP_7x7mm_P0.5mm_EP5.3x5.3mm
- removed QFN64: QFN-64-1EP_9x9mm_P0.5mm_EP3.4x3.4mm, Package_DFN_QFN:QFN-64-1EP_9x9mm_P0.5mm_EP3.4x3.4mm
- removed R1, R3: 5.1k, Resistor_SMD:R_0805_2012Metric_Pad1.20x1.40mm_HandSolder
- removed R2: 499, Resistor_SMD:R_0805_2012Metric_Pad1.20x1.40mm_HandSolder
- removed REF** (x3): KiCad-Logo2_5mm_SilkScreen, Symbol:KiCad-Logo2_5mm_SilkScreen
- removed SC-59: SC-59, Package_TO_SOT_SMD:SC-59
- removed SC-70: SC-70-8, Package_TO_SOT_SMD:SC-70-8
- removed SO-8: SO-8_3.9x4.9mm_P1.27mm, Package_SO:SO-8_3.9x4.9mm_P1.27mm
- removed SOT-89-5: SOT-89-5, Package_TO_SOT_SMD:SOT-89-5
- removed the SW38 at (59.9, 162.5)
- removed SW41: SW_Push, Switch_Keyboard_Kailh:SW_Kailh_Choc_V1V2_1.00u
- removed SW74: Left/Right, Jumper:SolderJumper-3_P1.3mm_Open_RoundedPad1.0x1.5mm_NumberLabels
- removed SW83: ~{RESET}, Button_Switch_SMD:SW_Tactile_SPST_NO_Straight_CK_PTS636Sx25SMTRLFS
- removed Scale: Gauge_10mm_Type2_CopperTop, Calibration_Scale:Gauge_10mm_Type2_CopperTop
- removed TP1: ROW_F, TestPoint:TestPoint_THTPad_1.5x1.5mm_Drill0.7mm
- removed TP10, TP7, TP8, TP9: SHIELD_POUR, TestPoint:TestPoint_THTPad_1.5x1.5mm_Drill0.7mm
- removed TP2: ROW_0, TestPoint:TestPoint_THTPad_1.5x1.5mm_Drill0.7mm
- removed TP3: ROW_1, TestPoint:TestPoint_THTPad_1.5x1.5mm_Drill0.7mm
- removed TP4: ROW_2, TestPoint:TestPoint_THTPad_1.5x1.5mm_Drill0.7mm
- removed TP5: ROW_3, TestPoint:TestPoint_THTPad_1.5x1.5mm_Drill0.7mm
- removed TP6: ROW_4, TestPoint:TestPoint_THTPad_1.5x1.5mm_Drill0.7mm
- removed U2: ATxmega32A4U-A, Package_QFP:TQFP-44_10x10mm_P0.8mm
- removed U3: USBLC6-2SC6, Package_TO_SOT_SMD:SOT-23-6
- removed VSON-10: VSON-10-1EP_3x3mm_P0.5mm_EP1.2x2mm, Package_SON:VSON-10-1EP_3x3mm_P0.5mm_EP1.2x2mm
- removed WSON-10: WSON-10-1EP_2.5x2.5mm_P0.5mm_EP1.2x2mm, Package_SON:WSON-10-1EP_2.5x2.5mm_P0.5mm_EP1.2x2mm
- SW1: renamed from SW45; value SW_Push -> F1
- SW2: renamed from SW46; value SW_Push -> F2
- SW3: renamed from SW47; value SW_Push -> f3
- SW4: renamed from SW48; value SW_Push -> F4
- SW5: renamed from SW49; value SW_Push -> F5
- SW6: renamed from SW50; value SW_Push -> F6
- SW7: renamed from SW51; value SW_Push -> F7
- U1: value MCP1700T-3302E_TT -> ~; footprint Package_TO_SOT_SMD:SOT-23 -> Adafruit_KB2040:KB2040; moved to B.Cu
- moved G*** 120.1 mm to (55.3, 170.1), turned to 180 degrees
- moved U1 67.3 mm to (80.4, 36.1), turned to 180 degrees
- renumbered D45 to D1, D12 to D10, D13 to D11, D14 to D12, D15 to D13, D16 to D14, D24 to D15, D18 to D16, D19 to D17, D20 to D18, D21 to D19, D46 to D2, D22 to D20, D23 to D21, D31 to D22, D25 to D23, D26 to D24, D27 to D25, D28 to D26, D29 to D27, D30 to D28, D39 to D29, D47 to D3, D32 to D30, D33 to D31, D34 to D32, D35 to D33, D36 to D34, D37 to D35, D40 to D36, D42 to D37, D43 to D38, D44 to D39, D48 to D4, D49 to D5, D50 to D6, D51 to D7, D17 to D8, D11 to D9, SW12 to SW10, SW13 to SW11, SW14 to SW12, SW15 to SW13, SW16 to SW14, SW24 to SW15, SW18 to SW16, SW19 to SW17, SW20 to SW18, SW21 to SW19, SW22 to SW20, SW23 to SW21, SW31 to SW22, SW25 to SW23, SW26 to SW24, SW27 to SW25, SW28 to SW26, SW29 to SW27, SW30 to SW28, SW39 to SW29, SW32 to SW30, SW33 to SW31, SW34 to SW32, SW35 to SW33, SW36 to SW34, SW37 to SW35, SW40 to SW36, SW42 to SW37, SW43 to SW38, SW44 to SW39, SW17 to SW8, SW11 to SW9
Connections:
- net /ROW_2 renamed /ROW_A
- net /ROW_3 renamed /ROW_Z
- D10 pad 1: /ROW_0 -> /ROW_1
- D11 pad 1: /ROW_0 -> /ROW_1
- D12 pad 1: /ROW_0 -> /ROW_1
- D13 pad 1: /ROW_0 -> /ROW_1
- D14 pad 1: /ROW_0 -> /ROW_1
- D15 pad 1: /ROW_1 -> /ROW_Q
- D16 pad 1: /ROW_1 -> /ROW_Q
- D17 pad 1: /ROW_1 -> /ROW_Q
- D18 pad 1: /ROW_1 -> /ROW_Q
- D19 pad 1: /ROW_1 -> /ROW_Q
- D20 pad 1: /ROW_1 -> /ROW_Q
- D21 pad 1: /ROW_1 -> /ROW_Q
- D36 pad 1: /ROW_4 -> /ROW_CMD
- D37 pad 1: /ROW_4 -> /ROW_CMD
- D38 pad 1: /ROW_4 -> Net-(D38-K)
- D39 pad 1: /ROW_4 -> Net-(D38-K)
- D8 pad 1: /ROW_0 -> /ROW_1
- D9 pad 1: /ROW_0 -> /ROW_1
- SW1 pad 1: /COL_1 -> /COL_0
- SW2 pad 1: /COL_2 -> /COL_1
- SW3 pad 1: /COL_3 -> /COL_2
- SW4 pad 1: /COL_4 -> /COL_3
- SW5 pad 1: /COL_5 -> /COL_4
- SW6 pad 1: /COL_6 -> /COL_5
- SW7 pad 1: /COL_0 -> /COL_6
- U1 pad 1: GND -> unconnected-(U1-USB_D+-Pad1)
- U1 pad 2: +3V3 -> unconnected-(U1-GPIO_0-Pad2)
- U1 pad 3: /VBUS_FUSED -> unconnected-(U1-GPIO_1-Pad3)
Routing:
- net /ROW_4: track 286.5 -> 0.00 mm, vias 3 -> 0
- net /ROW_Z: track 262.4 -> 0.00 mm, vias 3 -> 0
- net /ROW_A: track 229.2 -> 0.00 mm, vias 3 -> 0
- net /ROW_1: track 208.5 -> 0.00 mm, vias 3 -> 0
- net /ROW_0: track 188.0 -> 0.00 mm, vias 3 -> 0
- net /COL_0: track 182.2 -> 0.00 mm
- net /COL_6: track 171.1 -> 0.00 mm
- net /ROW_F: track 169.2 -> 0.00 mm, vias 1 -> 0
- net /COL_1: track 167.8 -> 0.00 mm
- net /COL_5: track 160.8 -> 0.00 mm
- net /COL_2: track 147.6 -> 0.00 mm
- net /COL_4: track 137.2 -> 0.00 mm
- net /COL_3: track 128.9 -> 0.00 mm
- net +3V3: track 70.4 -> 0.00 mm, vias 3 -> 0
- net /TXD0: track 57.4 -> 0.00 mm, vias 1 -> 0
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- removed copper zone on B.Cu, net /SHIELD_POUR
- removed copper zone on F.Cu, net /SHIELD_POUR
- removed copper zone on B.Cu, net GND
- removed copper zone on F.Cu, net GND
Other:
- board text added: "Copyright 2024, Revision 2"
- board text removed: "0.5mm"
- board text removed: "0.65mm"
- board text removed: "1.27"
- board text removed: "COL_1"
- board text removed: "Copyright 2023, Revision 1"
- board text removed: "LED"
- board text removed: "LEFT"
- board text removed: "R"
- board text removed: "Reset"
